File: src/sch/oggbox.sch (KiCad schematic (older format))
At the start: 145 parts

Commit message: Forgot to keep git up to date, loads of updates.
Parts:
- removed IC?: TC1016-1.8VC, symbol TC1016-1.8VC
- removed IC?: TC1016-2.8VC, symbol TC1016-2.8VC
- removed P?: CONN_10X2, symbol CONN_10X2
- removed P?: H/PHNS, symbol STEREO_JACK
- removed P?: LINE, symbol STEREO_JACK
- removed PWR? (x2): +2.8V, symbol +2.8V
- removed Q? (x2): NPN, symbol NPN
- removed Q? (x2): 2N3904, symbol 2N3904
- removed R? (x3): 10k, symbol R
- removed R? (x2): 33k, symbol R
- removed R? (x2): 470, symbol R
- removed SW?: UP, symbol SW_PUSH
- added C49, C50, C51, C52, C53, C54: 0.1u, symbol CS
- added C55: 0.1u, symbol C
- added IC7: TPS76318, symbol TPS76318
- added IC8: TPS76328, symbol TPS76328
- added IC9: MCP102, symbol MCP102
- added P10: HPHN, symbol CONN_4
- added P8: JTAG, symbol CONN_8
- added P9: LINE, symbol CONN_4
- added Q1, Q2: BC817, symbol BC817
- added Q3: BSH121, symbol BSH121
- added R39: 0, symbol R
- B1: renamed from B?; value CELL -> LIPO
- C1, C2: renamed from C?; value 18pF -> 18p
- C18, C20, C21: renamed from C?; value 0.01 -> 0.01u
- C19, C22: renamed from C?; value CAPAPOL -> 4.7u
- C23: renamed from C?; value 47uF -> 47u
- C24, C25: renamed from C?; value 10pF -> 10p
- C26, C30, C31, C38: renamed from C?; value 4.7uF -> 4.7u
- C27, C46: renamed from C?; value 100nF -> 0.1u
- C28, C29: renamed from C?; value 27pF -> 27p
- C39, C40, C41: renamed from C?; value 2.2uF -> 2.2u
- C43, C44: renamed from C?; value C -> 1u
- C45, C7: renamed from C?; value 0.1uF -> 0.1u
- C47, C48: renamed from C?; value C -> 4.7u; ESR (none) -> <10R
- C5, C6: renamed from C?; value .01u -> 0.01u
- L1: renamed from L?; value 470nH -> 470n
- L2, L3: renamed from L?; value 4.7uH -> 4.7u
- P2: renamed from P?; value CONN_6 -> USB
- R25: renamed from R?; value R -> 10k
- R37, R38: renamed from R?; value 2k -> 10k
- SW1, SW2, SW3, SW4, SW5, SW7, SW8, SW9: renamed from SW?; Farnell (none) -> 9962859
- SW10: renamed from SW?; value PWR -> UP; Farnell (none) -> 9962859
- gave numbers to parts that had none: 80
Connections:
- net labels added: +2.8V, A1, A2, K, Lx1, Lx2, SD_POW, VBAT, VOL_DN, VOL_UP
- net labels removed: SETBTN
- wire segments 524 -> 508
Other:
- moved on the sheet: C43, C44, L1, P5, R16, R32, R33, R34, R46, R52, R53, R54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

Commit message: More PCB routing, removed some unneccessary stuff and tidied up the charger circuit.  Bi colour LED now on the STM32 not VS1053
Parts:
- removed C31, C38: 4.7u, symbol CAPAPOL
- removed IC6: MCP1603T, symbol MCP1603T
- removed L3: 4.7u, symbol INDUCTOR
- added Q4: BSH121, symbol BSH121
- added R40, R43, R44: 10k, symbol R
- R35: value 2k -> 3k3
- R36: value 10k -> 12k
Connections:
- net labels added: CHG_FAST, VBAT_SENSE
- net labels removed: +3.3VP, CHG100, CHG500, Lx2, VBAT/2
- wire segments 508 -> 502
Other:
- moved on the sheet: C43, C44, D1, R11, R2
