File: sch/oggbox.kicad_pcb (KiCad board)
At the start: 4 copper layers, 100 x 50 mm, 169 parts, among them IC1 VS1053, IC2 MCP73831T, IC3 SD_CARD, IC4 MCP1802T-3002I-OT, IC5 STM32F103RET, IC6 MCP1802T-3002I-OT, IC7 TPS76318, IC8 TPS76328, IC9 MCP102, P1 CONN_3, P10 PHONES, P2 USB, P3 CORTEX_DEBUG, P4 CONN_1, P5 CONN_4, P6 CONN_28, P7 FTDI, P9 LINE, Q1 BSH121, Q2 BSH121, Q3 BSH121, Q4 BSH121, Q5 BSH121, Q6 BSS84AKW, SW1 VOL_UP, SW10 UP, SW11 HOLD, SW2 VOL_DN, SW3 RESET, SW4 MENU, SW5 SET, SW7 DOWN, SW8 LEFT, SW9 RIGHT, X1 12.288MHz, X2 32768Hz, X3 8MHz

Commit message: Updated the OggBox project to work with KiCad v5, made it a demo for automated manufacturing outputs
Parts:
- C1, C10, C11, C12, C13, C14, C15, C16, C17, C18, C2, C20, C21, C24, C25, C27, C28, C29, C3, C31, C32, C33, C34, C35, C36, C4, C42, C43, C44, C45, C46, C49, C5, C50, C51, C52, C53, C54, C55, C56, C57, C58, C59, C6, C60, C61, C7, C8, C9, R1, R10, R11, R12, R13, R14, R15, R16, R17, R18, R19, R2, R20, R21, R22, R23, R24, R25, R26, R27, R28, R29, R3, R30, R31, R32, R33, R34, R35, R36, R37, R38, R39, R4, R40, R41, R42, R43, R44, R45, R46, R47, R48, R49, R5, R50, R51, R52, R53, R54, R55, R56, R57, R58, R59, R6, R60, R61, R62, R63, R64, R65, R66, R67, R7, R8, R9: footprint SM0603 -> Nathan_SMT_Passive:SM0603
- C19, C22, C26, C30, C37, C38, C39, C40, C41, C47, C48, C62, C63: footprint SM0805 -> Nathan_SMT_Passive:SM0805
- C23, L1: footprint SM1206 -> Nathan_SMT_Passive:SM1206
- D1, IC9: footprint SOT23 -> Nathan_SMT_Semis:SOT23
- IC1: footprint LQFP48 -> Nathan_SMT_Semis:LQFP48
- IC2, IC4, IC6, IC7, IC8: footprint SOT23-5 -> Nathan_SMT_Semis:SOT23-5
- IC3: footprint SD_UNIVERSAL -> Nathan_SMT_Conn:SD_UNIVERSAL
- IC5: footprint LQFP64 -> Nathan_SMT_Semis:LQFP64
- P1: footprint JST_S3B_XHA -> Nathan_THT_Conn:JST_S3B_XHA
- P10, P9: footprint JACK_LUMBERG_1503_13_VP3 -> Nathan_SMT_Conn:JACK_LUMBERG_1503_13_VP3
- P2: footprint MICRO_USB_1568026 -> Nathan_SMT_Conn:MICRO_USB_1568026
- P3: footprint SAMTEC_SHF-SM_5x2 -> Nathan_SMT_Conn:SAMTEC_SHF-SM_5x2
- P4: footprint OSHW_COPPER_10MM -> Nathan_SMT_Other:OSHW_COPPER_10MM
- P5: footprint BTHQ128064AVD1 -> Nathan_THT_Other:BTHQ128064AVD1
- P6: footprint AMP_FPC_28_05MM -> Nathan_SMT_Conn:AMP_FPC_28_05MM
- P7: footprint HEADER_6 -> Nathan_THT_Conn:HEADER_6
- Q1, Q2, Q3, Q4, Q5, Q6: footprint SOT323 -> Nathan_SMT_Semis:SOT323
- SW1, SW2, SW3: footprint SW_SKQLLCE012 -> Nathan_SMT_Other:SW_SKQLLCE012
- SW10, SW4, SW5, SW7, SW8, SW9: footprint SW_EVQQ2P03W -> Nathan_SMT_Other:SW_EVQQ2P03W
- SW11: footprint PCM12SMTR -> Nathan_SMT_Other:PCM12SMTR
- X1: footprint CRYSTAL-SMD-5-3_2 -> Nathan_SMT_Other:CRYSTAL-SMD-5-3_2
- X2: footprint MC306 -> Nathan_SMT_Other:MC306
- X3: footprint XTAL_6036 -> Nathan_SMT_Other:XTAL_6036
